File: kicad/project.kicad_pcb (KiCad board)
At the start: 2 copper layers, 157.1 x 72.2 mm, 15 parts, among them J0 Conn_01x03_Female, U0 ProMicro here!

Commit message: 3d files
Other:
- outline, holes or cut-outs redrawn

Commit message: fix gerbers
Parts:
- moved ? 5.02 mm to (107.2, 96.8) (x2)
